File: hardware/10004_epic_cape.brd (EAGLE design)
At the start: 94 x 54.6 mm, 65 parts, among them J1 MSP430_BSL_HDR/SMD, SW1 KAS1102ET, SW2 KAS1102ET, U1 BEAGLEBONE_OUTLINE, U2 EPIC-CORE_A, U3 CAT24C256/SOIC-8, U4 MIC2025/SOIC-8

Commit message: Update design
Parts:
- removed U$1: (no value), frames:FRAME_A_L
- removed U$6: (no value), frames:DOCFIELD
- added C11: (no value), fcd:CAPC1005
- added J2: 5.5x2.1mm Barrel, SparkFun-Connectors:POWER_JACK_SMD
- added JP1: (no value), fcd:1X08
- added JP2, JP3, JP4: (no value), fcd:1X04
- added JP5: M07X2SHD_SMD, fcd:2X7-SHROUDED_SMD
- added R35, R36, R37, R38, R39, R40, R41, R42, R5, R52, R53, R54, R55, R57, R6, R7, R8: 0, fcd:RESC1005
- added R43, R44, R45, R46, R47, R48, R49, R50, R51: 10K, fcd:RESC1005
- added R56: (no value), fcd:RESC1005
- moved U$2 57.8 mm to (17.8, 40.0), turned to 0 degrees
- moved U$5 47.7 mm to (28.6, 7.62)
- moved U$4 40.2 mm to (24.8, 44.5)
- moved U$3 38.1 mm to (77.2, 7.62)
- moved C13 6.98 mm to (44.5, 33.0)
- moved J1 6.98 mm to (40.0, 27.3)
- moved C17 5.08 mm to (34.9, 14.0)
- moved R23 5.08 mm to (30.5, 19.7)
- moved U3 5.08 mm to (31.1, 14.0)
- moved R11 5.08 mm to (36.2, 14.0)
- moved R12 5.08 mm to (37.5, 14.0)
- moved R19 5.08 mm to (35.6, 19.7)
- moved R20 5.08 mm to (34.3, 19.7)
- moved R21 5.08 mm to (33.0, 19.7)
- moved R22 5.08 mm to (31.8, 19.7)
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Connections:
- net EPIC_RST/NMI_ST renamed BB_GPIO3_21
- net EPIC_TCK_ST renamed BB_GPIO1_17
- net EPIC_UART0RX_ST renamed BB_UART2_TXD
- net EPIC_UART0TX_ST renamed BB_UART2_RXD
- net EPIC_UART1RX_ST renamed BB_UART1_TXD
- net EPIC_UART1TX_ST renamed BB_UART1_RXD
- net PWR_EN_ST renamed BB_GPIO1_16
- net PWR_FLG_ST renamed BB_GPIO1_28
- removed net GPIO2_6: U1.45
- removed net GPIO2_7: U1.46
- removed net GPIO2_8: U1.43
- removed net GPIO2_9: U1.44
- new net BB_GPIO2_6: R39.2, U1.45
- new net BB_GPIO2_7: R40.2, U1.46
- new net BB_GPIO2_8: R41.2, U1.43
- new net BB_GPIO2_9: R42.2, U1.44
- new net BB_SPI1_CS0: R5.2, U1.74
- new net BB_SPI1_DI: R6.2, U1.76
- new net BB_SPI1_DO: R7.2, U1.75
- new net BB_SPI1_SCLK: R8.2, U1.77
- new net EPIC_ADC0: JP2.1, U2.P$19
- new net EPIC_ADC1: JP3.1, U2.P$20
- new net EPIC_ADC2: JP2.2, U2.P$21
- new net EPIC_ADC3: JP3.2, U2.P$22
- new net EPIC_ADC4: JP2.3, U2.P$23
- new net EPIC_ADC5: JP3.3, U2.P$24
- new net EPIC_ADC6: JP2.4, U2.P$25
- new net EPIC_ADC7: JP3.4, U2.P$26
- new net EPIC_MISO1: JP1.3, R37.1, R7.1
- new net EPIC_MISO1_ST: R37.2, U2.P$4
- new net EPIC_MOSI1: JP1.2, R36.1, R6.1
- new net EPIC_MOSI1_ST: R36.2, U2.P$3
- new net EPIC_P1.2: JP4.1, R43.1, U2.P$30
- new net EPIC_P1.5: JP4.2, R44.1, U2.P$31
- new net EPIC_P1.6: JP4.3, R45.1, U2.P$32
- new net EPIC_P1.7: JP4.4, R46.1, U2.P$33
- new net EPIC_P2.0: R42.1, R50.1, U2.P$38
- new net EPIC_P2.1: R41.1, R49.1, U2.P$39
- new net EPIC_P2.3: R40.1, R48.1, U2.P$40
- new net EPIC_P2.6: R39.1, R47.1, U2.P$41
- new net EPIC_P5.4: JP1.5, U2.P$6
- new net EPIC_P5.5: JP1.6, U2.P$7
- new net EPIC_P5.6: JP1.7, U2.P$8
- new net EPIC_P5.7: JP1.8, U2.P$9
- new net EPIC_SCLK1: JP1.4, R38.1, R8.1
- new net EPIC_SCLK1_ST: R38.2, U2.P$5
- new net EPIC_STE1: JP1.1, R35.1, R5.1
- new net EPIC_STE1_ST: R35.2, U2.P$2
- new net EPIC_TDI/TCLK: JP5.3, U2.P$13
- new net EPIC_TDO/TDI: JP5.1, U2.P$12
- new net EPIC_TMS: JP5.5, U2.P$14
- new net N$18: JP5.12, R52.1
- new net N$20: JP5.14, R53.1
- new net N$3: JP5.13, R54.2
- new net VCCTARGET: JP5.4, R57.1
- new net VCCTOOL: JP5.2, R55.1
- net 3V3: now also J2.VIN0, R43.2, R44.2, R45.2, R46.2, R47.2, R48.2, R49.2, R50.2, R55.2, R56.2, R57.2, R9.2; no longer R25.2
- net EPIC_RST/NMI: now also C11.1, JP5.11, R56.1
- net EPIC_TCK: now also JP5.7
- net EPIC_UART1RX: now also R53.2
- net EPIC_UART1TX: now also R52.2
- net GND: now also C11.2, J2.GND, J2.P$4, JP5.9, R51.1, R54.1
- net PWR_EN: now also R51.2
- net VDD_3V3EXP: now also R25.2; no longer R9.2
Routing:
- net EPIC_STE1: track 0.00 -> 36.4 mm
- net EPIC_MOSI1: track 0.00 -> 35.1 mm
- net 3V3: track 46.2 -> 80.7 mm, vias 20 -> 28
- net EPIC_UART1TX: track 48.2 -> 81.8 mm, vias 2 -> 3
- net EPIC_UART1RX: track 51.8 -> 84.7 mm, vias 2 -> 3
- net EPIC_P2.0: track 0.00 -> 32.8 mm, vias 0 -> 2
- net EPIC_MISO1: track 0.00 -> 32.7 mm
- net EPIC_SCLK1: track 0.00 -> 31.4 mm
- net EPIC_P2.1: track 0.00 -> 30.5 mm, vias 0 -> 2
- net EPIC_RST/NMI: track 79.4 -> 107.6 mm, vias 5 -> 4
- net EPIC_P2.3: track 0.00 -> 28.2 mm, vias 0 -> 2
- net EPIC_P2.6: track 0.00 -> 26.9 mm, vias 0 -> 2
- net VCCTARGET: track 0.00 -> 23.1 mm
- net EPIC_TCK: track 23.8 -> 45.0 mm, vias 2 -> 3
- net GND: track 93.4 -> 111.4 mm, vias 34 -> 44
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- added copper zone on layer 1, net GND
Other:
- board text removed: "1.1.1"
- board text removed: "Epic Cape for BeagleBone"
- board text removed: "Flying Camp Design - www.flyingcampdesign.com"
