File: hardware/10004_epic_cape.sch (EAGLE design)
At the start: 63 parts, among them J1 MSP430_BSL_HDR/SMD, SW1 KAS1102ET, SW2 KAS1102ET, U1 BEAGLEBONE_OUTLINE, U2 EPIC-CORE_A, U3 CAT24C256/SOIC-8, U4 MIC2025/SOIC-8

Commit message: Update design
Parts:
- added C11: (no value), fcd:CAPACITOR1005
- added J2: 5.5x2.1mm Barrel, SparkFun-Connectors:POWER_JACKSMD
- added JP1: (no value), fcd:M081X08
- added JP2, JP3, JP4: (no value), fcd:M04PTH
- added JP5: M07X2SHD_SMD, fcd:M07X2SHD_SMD
- added R35, R36, R37, R38, R39, R40, R41, R42, R5, R52, R53, R54, R55, R57, R6, R7, R8: 0, fcd:RESISTOR1005
- added R43, R44, R45, R46, R47, R48, R49, R50, R51: 10K, fcd:RESISTOR1005
- added R56: (no value), fcd:RESISTOR1005
Connections:
- net EPIC_RST/NMI_ST renamed BB_GPIO3_21
- net EPIC_TCK_ST renamed BB_GPIO1_17
- net EPIC_UART0RX_ST renamed BB_UART2_TXD
- net EPIC_UART0TX_ST renamed BB_UART2_RXD
- net EPIC_UART1RX_ST renamed BB_UART1_TXD
- net EPIC_UART1TX_ST renamed BB_UART1_RXD
- net PWR_EN_ST renamed BB_GPIO1_16
- net PWR_FLG_ST renamed BB_GPIO1_28
- new net BB_GPIO2_6: R39.2, U1.GPIO2_6
- new net BB_GPIO2_7: R40.2, U1.GPIO2_7
- new net BB_GPIO2_8: R41.2, U1.GPIO2_8
- new net BB_GPIO2_9: R42.2, U1.GPIO2_9
- new net BB_SPI1_CS0: R5.2, U1.SPI1_CS0
- new net BB_SPI1_DI: R6.2, U1.SPI1_DI
- new net BB_SPI1_DO: R7.2, U1.SPI1_DO
- new net BB_SPI1_SCLK: R8.2, U1.SPI1_SCLK
- new net EPIC_ADC0: JP2.1, U2.ADC0
- new net EPIC_ADC1: JP3.1, U2.ADC1
- new net EPIC_ADC2: JP2.2, U2.ADC2
- new net EPIC_ADC3: JP3.2, U2.ADC3
- new net EPIC_ADC4: JP2.3, U2.ADC4
- new net EPIC_ADC5: JP3.3, U2.ADC5
- new net EPIC_ADC6: JP2.4, U2.ADC6/DAC0
- new net EPIC_ADC7: JP3.4, U2.ADC7/DAC1
- new net EPIC_MISO1: JP1.3, R37.1, R7.1
- new net EPIC_MISO1_ST: R37.2, U2.P5.2
- new net EPIC_MOSI1: JP1.2, R36.1, R6.1
- new net EPIC_MOSI1_ST: R36.2, U2.P5.1
- new net EPIC_P1.2: JP4.1, R43.1, U2.P1.2
- new net EPIC_P1.5: JP4.2, R44.1, U2.P1.5
- new net EPIC_P1.6: JP4.3, R45.1, U2.P1.6
- new net EPIC_P1.7: JP4.4, R46.1, U2.P1.7
- new net EPIC_P2.0: R42.1, R50.1, U2.P2.0
- new net EPIC_P2.1: R41.1, R49.1, U2.P2.1
- new net EPIC_P2.3: R40.1, R48.1, U2.P2.3
- new net EPIC_P2.6: R39.1, R47.1, U2.P2.6
- new net EPIC_P5.4: JP1.5, U2.P5.4
- new net EPIC_P5.5: JP1.6, U2.P5.5
- new net EPIC_P5.6: JP1.7, U2.P5.6
- new net EPIC_P5.7: JP1.8, U2.P5.7
- new net EPIC_SCLK1: JP1.4, R38.1, R8.1
- new net EPIC_SCLK1_ST: R38.2, U2.P5.3
- new net EPIC_STE1: JP1.1, R35.1, R5.1
- new net EPIC_STE1_ST: R35.2, U2.P5.0
- new net EPIC_TDI/TCLK: JP5.3, U2.TDI/TCLK
- new net EPIC_TDO/TDI: JP5.1, U2.TDO/TDI
- new net EPIC_TMS: JP5.5, U2.TMS
- new net N$18: JP5.12, R52.1
- new net N$20: JP5.14, R53.1
- new net N$3: JP5.13, R54.2
- new net VCCTARGET: JP5.4, R57.1
- new net VCCTOOL: JP5.2, R55.1
- net 3V3: now also J2.PWR, R43.2, R44.2, R45.2, R46.2, R47.2, R48.2, R49.2, R50.2, R55.2, R56.2, R57.2, R9.2; no longer R25.2
- net EPIC_RST/NMI: now also C11.1, JP5.11, R56.1
- net EPIC_TCK: now also JP5.7
- net EPIC_UART1RX: now also R53.2
- net EPIC_UART1TX: now also R52.2
- net GND: now also C11.2, J2.GND, J2.GNDBREAK, JP5.9, R51.1, R54.1
- net PWR_EN: now also R51.2
- net VDD_3V3EXP: now also R25.2; no longer R9.2
Other:
- note added: "BEAGLEBONE HEADERS"
- note added: "EEPROM & DIP SWITCHES & POWER INPUT & JTAG"
- note removed: "BEAGLEBONE HEADERS & POWER SWITCH"
- note removed: "EEPROM & CONFIG SWITCHES"
