File: hardware/10004_epic_cape/10004_epic_cape.brd (EAGLE design)
At the start: 94 x 54.6 mm, 97 parts, among them J1 MSP430_BSL_HDR/SMD, J2 5.5x2.1mm Barrel, SW1 KAS1102ET, SW2 KAS1102ET, U1 BEAGLEBONE_OUTLINE, U2 EPIC-CORE_A, U3 CAT24C256/SOIC-8, U4 MIC2025/SOIC-8

Commit message: Release 1.1.1
Parts:
- added BT1: KEYSTONE_2462, fcd:KEYSTONE_2462
- added JP6: M02PTH, fcd:1X02
- moved U$3 0.32 mm to (77.2, 7.94)
Connections:
- net 3V3: now also BT1.+, JP6.1
- net GND: now also BT1.-, JP6.2
Routing:
- net CAPE_EEPROM_A1: track 14.0 -> 20.8 mm
- net GND: track 111.4 -> 117.5 mm, vias 44 -> 45
- net RFGND: track 0.00 -> 2.44 mm
- net BB_I2C2_SDA: track 18.9 -> 20.3 mm
- net BB_I2C2_SCL: track 15.5 -> 16.2 mm
- net CAPE_EEPROM_A0: track 11.9 -> 12.6 mm
