File: hardware/10004_epic_cape/10004_epic_cape.sch (EAGLE design)
At the start: 97 parts, among them J1 MSP430_BSL_HDR/SMD, J2 5.5x2.1mm Barrel, SW1 KAS1102ET, SW2 KAS1102ET, U1 BEAGLEBONE_OUTLINE, U2 EPIC-CORE_A, U3 CAT24C256/SOIC-8, U4 MIC2025/SOIC-8

Commit message: Release 1.1.1
Parts:
- added BT1: KEYSTONE_2462, fcd:KEYSTONE_2462
- added JP6: M02PTH, fcd:M02PTH
- J2: COST (none) -> 1.12100; MFR (none) -> CUI; MPN (none) -> PJ-002AH-SMT-TR
Connections:
- net 3V3: now also BT1.+, JP6.1
- net GND: now also BT1.-, JP6.2
Other:
- note added: "8-BIT GPIO"
- note added: "AA BATTERY HOLDER FOR STANDALONE MODE"
- note added: "ADC INPUTS"
- note added: "BEAGLEBONE CAPE EEPROM"
- note added: "DC INPUT FOR STANDALONE MODE"
- note added: "EEPROM / FLASH WRITE PROTECT SWITCH"
- note added: "INTERRUPTIBLE GPIO"
- note added: "MSP430 JTAG & BSL HEADER"
- note added: "POWER DISTRIBUTION SWITCH 500MA MAX"
- moved on the sheet: C15, C16, C17, J2, JP1, JP4, R10, R19, R20, R21, R22, R23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
